File: hardware/luluu.kicad_pcb (KiCad board)
At the start: 4 copper layers, 64.1 x 30 mm, 57 parts, among them J1 BATT_CON, J2 RPi SWD, J3 STEMMA_{QT} I_{2}C, J4 Micro_SD_Card, J6 USB_C_Receptacle_USB2.0, J7 DISP_LCD_ST7789, Q1 AO3401A, Q2 BSS138, SW1 SW_USBBOOT, SW2 SW_RESET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

Commit message: more work on v2.0
Parts:
- added J5: GPIO0, Connector_PinHeader_2.54mm:PinHeader_1x05_P2.54mm_Vertical, F.Cu at (122.5, 79.7)
- added J8: GPIO1, Connector_PinHeader_2.54mm:PinHeader_1x07_P2.54mm_Vertical, F.Cu at (143.8, 105.2)
- added MNT0: Pin_D1.0mm_L10.0mm, Connector_Pin:Pin_D1.0mm_L10.0mm, F.Cu at (112.5, 105.2)
- added MNT1: Pin_D1.0mm_L10.0mm, Connector_Pin:Pin_D1.0mm_L10.0mm, F.Cu at (171.5, 79.8)
- added MNT2: Pin_D1.0mm_L10.0mm, Connector_Pin:Pin_D1.0mm_L10.0mm, F.Cu at (162.0, 105.2)
- moved C20 5.23 mm to (113.8, 83.0), turned to 180 degrees
- moved J3 2.23 mm to (113.5, 100.5)
- moved R14 1.34 mm to (119.0, 105.0), turned to -90 degrees
- moved C16 1.18 mm to (133.2, 94.7)
- moved C17 0.99 mm to (132.4, 105.5)
- moved R15 0.94 mm to (122.8, 82.8), turned to 180 degrees
- moved C19 0.92 mm to (138.3, 105.4)
- moved Q2 0.84 mm to (124.0, 86.0)
- moved R13 0.84 mm to (124.0, 90.8)
- moved R9 0.84 mm to (124.0, 89.0)
- moved J7 0.82 mm to (115.6, 90.2)
- moved Q1 0.80 mm to (161.1, 91.2)
- moved C1 0.80 mm to (147.6, 96.5)
- moved C10 0.80 mm to (141.9, 98.8)
- moved C11 0.80 mm to (128.4, 101.7)
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Connections:
- U3 pad 11: unconnected-(U3-GPIO8-Pad11) -> /GPIO_D8
- U3 pad 12: unconnected-(U3-GPIO9-Pad12) -> /GPIO_D9
- U3 pad 15: unconnected-(U3-GPIO12-Pad15) -> /GPIO_D12
- U3 pad 36: unconnected-(U3-GPIO24-Pad36) -> /GPIO_D24
- U3 pad 37: unconnected-(U3-GPIO25-Pad37) -> /GPIO_D25
- U3 pad 38: unconnected-(U3-GPIO26_ADC0-Pad38) -> /GPIO_A0
- U3 pad 39: unconnected-(U3-GPIO27_ADC1-Pad39) -> /GPIO_A1
- U3 pad 40: unconnected-(U3-GPIO28_ADC2-Pad40) -> /GPIO_A2
- U3 pad 9: unconnected-(U3-GPIO7-Pad9) -> /GPIO_D7
Routing:
- net /GPIO_D12: track 0.00 -> 31.9 mm, vias 0 -> 1
- net /GPIO_D9: track 0.00 -> 28.1 mm, vias 0 -> 1
- net /GPIO_D8: track 0.00 -> 26.2 mm, vias 0 -> 1
- net /GPIO_D7: track 0.00 -> 24.8 mm, vias 0 -> 1
- net /GPIO_D24: track 0.00 -> 22.5 mm, vias 0 -> 1
- net /GPIO_D25: track 0.00 -> 20.4 mm, vias 0 -> 1
- net /GPIO_A0: track 0.00 -> 16.6 mm, vias 0 -> 1
- net /GPIO_A1: track 0.00 -> 12.5 mm, vias 0 -> 1
- net /GPIO_A2: track 0.00 -> 8.66 mm, vias 0 -> 1
- net GND: track 106.0 -> 99.7 mm
- net +3V3: track 266.1 -> 269.8 mm
- net /SWD: track 28.1 -> 27.1 mm
- net /I_{2}C_{CLOCK}: track 23.5 -> 24.2 mm
- net Net-(J7-BACKLIGHT_{K}): track 7.02 -> 7.70 mm
- net /DISP_~{CS_{MAIN}}: track 37.1 -> 37.7 mm
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- removed copper zone on B.Cu, net +3V3
- removed copper zone on F.Cu, net +3V3
Other:
- board size 64.1 x 30 mm -> 64 x 30 mm
- board text added: "12"
- board text added: "24"
- board text added: "25"
- board text added: "3v3"
- board text added: "7"
- board text added: "8"
- board text added: "9"
- board text added: "A0"
- board text added: "A1"
- board text added: "A2"
- board text added: "GND"
- board text removed: "by gray olson"
- board text removed: "made with <3"
